Commit message: update

File: catkin_ws/src/smartcar_description/src/smartcar_description/urdf/smartcar (another copy).urdf (robot description, URDF)
Before this commit: robot origins, 12 links, 11 joints
Links:
- link left_gripper: geometry collision box size=0.1 .1 .1; visual mesh filename=package://pr2_description/meshes/gripper_v0/l_finger.dae
- link left_tip: geometry collision box size=0.1 .1 .1; visual mesh filename=package://pr2_description/meshes/gripper_v0/l_finger_tip.dae
- link right_gripper: geometry collision box size=0.1 .1 .1; visual mesh filename=package://pr2_description/meshes/gripper_v0/l_finger.dae
- link right_tip: geometry collision box size=0.1 .1 .1; visual mesh filename=package://pr2_description/meshes/gripper_v0/l_finger_tip.dae
